File: chargerV1.kicad_sch (KiCad schematic)
At the start: 46 parts, among them J1 USB_C_Receptacle, J2 SOCKET_1x4, J3 SOCKET_1x4, J4 SOCKET_1x6, J5 Micro_SD_Card, SW1 BOOT, SW2 OK, SW3 RESET, SW4 UP, SW5 DW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

Commit message: Add modifies
Parts:
- C14, C15, C16, C17, C24: footprint IVSFootprint:C0603 -> IVS_footprints:C_0603
- J2, J3, SENSOR1: footprint IVSFootprint:SH-1.0mm-1x4 -> IVS_footprints:JST_SH_SM04B-SRSS-TB_1x04-1MP_P1.00mm_Horizontal
- J4: footprint IVSFootprint:SH-1.0mm-1x6 -> IVS_footprints:JST_SH_SM06B-SRSS-TB_1x06-1MP_P1.00mm_Horizontal
- LCD1: footprint IVSFootprint:SH-1.0mm-1x8 -> IVS_footprints:JST_SH_SM08B-SRSS-TB_1x08-1MP_P1.00mm_Horizontal
- SW1, SW3: footprint IVSFootprint:SW_SPST_PTS810 -> IVS_footprints:SW_SPST_PTS810
- SW2, SW4, SW5: footprint IVS_footprints:BUTTON_PUSH_12mm -> IVS_footprints:Button_Push_12mm
Other:
- moved on the sheet: C14, C15, C16, C17, LE1, R4, U4

Commit message: Add more modifies
Parts:
- C4, C6, C7, C8: footprint IVSFootprint:C0603 -> IVS_footprints:C_0603
- D1: footprint IVSFootprint:D_MiniMELF -> IVS_footprints:D_MiniMELF
Changed lines of the file:
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@@
       (effects (font (size 1.27 1.27)) (justify left))
     )
-    (property "Footprint" "IVSFootprint:C0603" (at 60.6552 175.26 0)
+    (property "Footprint" "IVS_footprints:C_0603" (at 60.6552 175.26 0)
       (effects (font (size 1.27 1.27)) hide)
     )
@@
       (effects (font (size 1.27 1.27)) (justify left))
     )
-    (property "Footprint" "IVSFootprint:C0603" (at 50.4952 175.26 0)
+    (property "Footprint" "IVS_footprints:C_0603" (at 50.4952 175.26 0)
       (effects (font (size 1.27 1.27)) hide)
     )
@@
       (effects (font (size 1.27 1.27)) (justify left))
     )
-    (property "Footprint" "IVSFootprint:C0603" (at 80.9752 175.26 0)
+    (property "Footprint" "IVS_footprints:C_0603" (at 80.9752 175.26 0)
       (effects (font (size 1.27 1.27)) hide)
     )
@@
       (effects (font (size 1.27 1.27)) (justify left))
     )
-    (property "Footprint" "IVSFootprint:D_MiniMELF" (at 40.64 171.45 0)
+    (property "Footprint" "IVS_footprints:D_MiniMELF" (at 40.64 171.45 0)
       (effects (font (size 1.27 1.27)) hide)
     )
@@
       (effects (font (size 1.27 1.27)) (justify left))
     )
-    (property "Footprint" "IVSFootprint:C0603" (at 70.8152 175.26 0)
-      (effects (font (size 1.27 1.27)) hide)
-    )
+    (property "Footprint" "IVS_footprints:C_0603" (at 70.8152 175.26 0)
+      (effects (font (size 1.27 1.27)) hide)
+    )

Commit message: Add more modifies
Parts:
- added C10: 10uF, IVS_footprints:C_0603, symbol Device:C
Connections:
- net GND: now also C10.2
- net VBUS: now also C10.1
Changed lines of the file:
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@@
   (junction (at 57.15 223.52) (diameter 0) (color 0 0 0 0)
   )
+  (junction (at 234.95 149.86) (diameter 0) (color 0 0 0 0)
+  )
   (junction (at 69.85 165.1) (diameter 0) (color 0 0 0 0)
   )
@@
   )
   (junction (at 53.34 223.52) (diameter 0) (color 0 0 0 0)
+  )
+  (junction (at 237.49 160.02) (diameter 0) (color 0 0 0 0)
   )
   (junction (at 207.01 78.74) (diameter 0) (color 0 0 0 0)
@@
     (stroke (width 0) (type default))
   )
+  (wire (pts (xy 240.03 160.02) (xy 237.49 160.02))
+    (stroke (width 0) (type default))
+  )
   (wire (pts (xy 69.85 328.93) (xy 69.85 335.788))
     (stroke (width 0) (type default))
@@
     (stroke (width 0) (type default))
   )
+  (wire (pts (xy 217.17 156.21) (xy 234.95 156.21))
+    (stroke (width 0) (type default))
+  )
+  (wire (pts (xy 234.95 149.86) (xy 234.95 147.32))
+    (stroke (width 0) (type default))
+  )
   (polyline (pts (xy 262.89 242.824) (xy 262.89 186.69))
     (stroke (width 0) (type default))
@@
   )
   (wire (pts (xy 58.42 267.97) (xy 58.42 273.05))
+    (stroke (width 0) (type default))
+  )
+  (wire (pts (xy 234.95 156.21) (xy 234.95 149.86))
     (stroke (width 0) (type default))
   )
@@
     (stroke (width 0) (type default) (color 0 255 0 1))
   )
+  (wire (pts (xy 240.03 158.75) (xy 240.03 160.02))
+    (stroke (width 0) (type default))
+  )
   (wire (pts (xy 140.97 106.68) (xy 158.75 106.68))
+    (stroke (width 0) (type default))
+  )
+  (wire (pts (xy 237.49 158.75) (xy 217.17 158.75))
     (stroke (width 0) (type default))
   )
@@
     (stroke (width 0) (type default))
   )
+  (wire (pts (xy 240.03 151.13) (xy 240.03 149.86))
+    (stroke (width 0) (type default))
+  )
   (wire (pts (xy 44.45 328.93) (xy 44.45 330.2))
     (stroke (width 0) (type default))
@@
     (stroke (width 0) (type default))
   )
-  (wire (pts (xy 217.17 156.21) (xy 226.06 156.21))
-    (stroke (width 0) (type default))
-  )
   (polyline (pts (xy 132.08 204.47) (xy 157.48 204.47))
     (stroke (width 0) (type default) (color 255 0 0 1))
@@
     (stroke (width 0) (type default))
   )
+  (wire (pts (xy 237.49 160.02) (xy 237.49 158.75))
+    (stroke (width 0) (type default))
+  )
   (wire (pts (xy 133.35 167.64) (xy 114.3 167.64))
     (stroke (width 0) (type default))
@@
     (stroke (width 0) (type default))
   )
+  (wire (pts (xy 240.03 149.86) (xy 234.95 149.86))
+    (stroke (width 0) (type default))
+  )
   (wire (pts (xy 73.66 262.89) (xy 73.66 266.7))
     (stroke (width 0) (type default))
@@
   )
   (wire (pts (xy 49.53 165.1) (xy 59.69 165.1))
-    (stroke (width 0) (type default))
-  )
-  (wire (pts (xy 217.17 158.75) (xy 231.14 158.75))
     (stroke (width 0) (type default))
   )
@@
   )
   (wire (pts (xy 57.15 209.55) (xy 57.15 213.36))
+    (stroke (width 0) (type default))
+  )
+  (wire (pts (xy 237.49 161.29) (xy 237.49 160.02))
     (stroke (width 0) (type default))
   )
@@
     )
   )
+  (symbol (lib_id "Device:C") (at 240.03 154.94 0) (unit 1)
+    (in_bom yes) (on_board yes) (dnp no)
+    (property "Reference" "C10" (at 243.84 153.6699 0)
+      (effects (font (size 1.27 1.27)) (justify left))
+    )
+    (property "Value" "10uF" (at 243.84 156.2099 0)
+      (effects (font (size 1.27 1.27)) (justify left))
+    )
+    (property "Footprint" "IVS_footprints:C_0603" (at 240.9952 158.75 0)
+      (effects (font (size 1.27 1.27)) hide)
+    )
+    (property "Datasheet" "~" (at 240.03 154.94 0)
+      (effects (font (size 1.27 1.27)) hide)
+    )
+    (pin "1")
+    (pin "2")
+    (instances
+      (project "chargerV1"
+        (path "/696df81d-5a87-441a-8d24-56d9edd75190"
+          (reference "C10") (unit 1)
+        )
+      )
+    )
+  )
   (symbol (lib_id "Device:C") (at 162.56 104.14 0) (unit 1)
     (in_bom yes) (on_board yes) (dnp no) (fields_autoplaced)
@@
     )
   )
-  (symbol (lib_id "power:GND") (at 231.14 158.75 90) (unit 1)
-    (in_bom yes) (on_board yes) (dnp no) (fields_autoplaced)
-    (property "Reference" "#PWR0123" (at 237.49 158.75 0)
-      (effects (font (size 1.27 1.27)) hide)
-    )
-    (property "Value" "GND" (at 234.95 159.385 90)
-      (effects (font (size 1.27 1.27)) (justify right))
-    )
-    (property "Footprint" "" (at 231.14 158.75 0)
-      (effects (font (size 1.27 1.27)) hide)
-    )
-    (property "Datasheet" "" (at 231.14 158.75 0)
+  (symbol (lib_id "power:GND") (at 237.49 161.29 0) (unit 1)
+    (in_bom yes) (on_board yes) (dnp no) (fields_autoplaced)
+    (property "Reference" "#PWR0123" (at 237.49 167.64 0)
+      (effects (font (size 1.27 1.27)) hide)
+    )
+    (property "Value" "GND" (at 240.03 163.195 0)
+      (effects (font (size 1.27 1.27)) (justify left))
+    )
+    (property "Footprint" "" (at 237.49 161.29 0)
+      (effects (font (size 1.27 1.27)) hide)
+    )
+    (property "Datasheet" "" (at 237.49 161.29 0)
       (effects (font (size 1.27 1.27)) hide)
     )
@@
     )
   )
-  (symbol (lib_id "power:VBUS") (at 226.06 156.21 270) (unit 1)
-    (in_bom yes) (on_board yes) (dnp no) (fields_autoplaced)
-    (property "Reference" "#PWR02" (at 222.25 156.21 0)
-      (effects (font (size 1.27 1.27)) hide)
-    )
-    (property "Value" "VBUS" (at 229.87 156.845 90)
-      (effects (font (size 1.27 1.27)) (justify left))
-    )
-    (property "Footprint" "" (at 226.06 156.21 0)
-      (effects (font (size 1.27 1.27)) hide)
-    )
-    (property "Datasheet" "" (at 226.06 156.21 0)
-      (effects (font (size 1.27 1.27)) hide)
-    )
+  (symbol (lib_id "power:VBUS") (at 234.95 147.32 0) (unit 1)
+    (in_bom yes) (on_board yes) (dnp no) (fields_autoplaced)
+    (property "Reference" "#PWR02" (at 234.95 151.13 0)
+      (effects (font (size 1.27 1.27)) hide)
+    )
+    (property "Value" "VBUS" (at 237.49 146.685 0)
+      (effects (font (size 1.27 1.27)) (justify left))
+    )
+    (property "Footprint" "" (at 234.95 147.32 0)
+      (effects (font (size 1.27 1.27)) hide)
+    )
+    (property "Datasheet" "" (at 234.95 147.32 0)
+      (effects (font (size 1.27 1.27)) hide)
+    )

Commit message: Fix buttons
Parts:
- removed J2, J3: SOCKET_1x4, IVS_footprints:JST_SH_SM04B-SRSS-TB_1x04-1MP_P1.00mm_Horizontal, symbol IVS_symbol:SOCKET_1x4
- removed SW2: OK, IVS_footprints:Button_Push_12mm, symbol IVS_SYMBOL:switch
- removed SW4: UP, IVS_footprints:Button_Push_12mm, symbol IVS_SYMBOL:switch
- removed SW5: DW, IVS_footprints:Button_Push_12mm, symbol IVS_SYMBOL:switch
- added P1: ~, IVS_footprints:JST_SH_SM05B-SRSS-TB_1x05-1MP_P1.00mm_Horizontal, symbol IVS_symbols:SOCKET_1x5
Connections:
- net +3.3V: now also P1.1
- net BUTT_DW: now also P1.3
- net BUTT_OK: now also P1.5
- net BUTT_UP: now also P1.4
- net GND: now also P1.2
Other:
- moved on the sheet: BT1, C1, C2, C24, C3, C4, C5, C6, C7, C8, D1, D2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
